Commit message: add actions

File: src/my_robot_description/urdf/my_robot.urdf.xacro (robot description, xacro)
@@ -4,3 +4,4 @@
     <xacro:include filename="simple_robot_car.urdf.xacro"/>
     <xacro:include filename="simple_robot_car_gazebo.urdf.xacro"/>
+    <xacro:include filename="camera.xacro"/>
 </robot>

File: src/my_robot_description/urdf/simple_robot_car.urdf.xacro (robot description, xacro)
@@ -1,6 +1,6 @@
 <?xml version="1.0"?>
 <robot xmlns:xacro="http://www.ros.org/wiki/xacro">
-    <xacro:property name="base_length" value="1.0" />
-    <xacro:property name="base_width" value="0.6" />
+    <xacro:property name="base_length" value="0.6" />
+    <xacro:property name="base_width" value="0.4" />
     <xacro:property name="base_height" value="0.2" />
     <xacro:property name="wheel_radius" value="0.1" />
@@ -21,5 +21,5 @@
                 <origin xyz="0 0 0" rpy="${pi / 2.0} 0 0" />
             </collision>
-            <xacro:cylinder_inertia m="1.0" r="${wheel_radius}" h="${wheel_length}" xyz="0 0 0" rpy="${pi / 2.0} 0 0" />
+            <xacro:cylinder_inertia m="1.0" r="${2*wheel_radius}" h="${2*wheel_length}" xyz="0 0 0" rpy="${pi / 2.0} 0 0" />
         </link>
     </xacro:macro>
@@ -40,5 +40,5 @@
             <origin xyz="0 0 ${base_height / 2.0}" rpy="0 0 0"></origin>
         </collision>
-        <xacro:box_inertia  m="5.0" l="${base_length}" w="${base_width}"  h="${base_height}"
+        <xacro:box_inertia  m="5.0" l="${2*base_length}" w="${2*base_width}"  h="${2*base_height}"
                             xyz="0 0 ${base_height / 2.0}" rpy="0 0 0" />
     </link>
@@ -59,5 +59,5 @@
             <origin xyz="0 0 0" rpy="0 0 0" />
         </collision>
-        <xacro:sphere_inertia   m="0.5" r="${wheel_radius / 2.0}"
+        <xacro:sphere_inertia   m="0.5" r="${2*wheel_radius / 2.0}"
                                 xyz="0 0 0" rpy="0 0 0" />
     </link>

File: src/my_robot_description/urdf/simple_robot_car_gazebo.urdf.xacro (robot description, xacro)
@@ -4,3 +4,35 @@
         <material>Gazebo/Blue</material>
     </gazebo>
+    <gazebo reference="right_wheel_link">
+        <material>Gazebo/Green</material>
+    </gazebo>
+    <gazebo reference="left_wheel_link">
+        <material>Gazebo/Green</material>
+    </gazebo>
+    <gazebo reference="caster_wheel_link">
+        <material>Gazebo/Grey</material>
+        <mu1 value="0.1"/>
+        <mu2 value="0.1"/>
+    </gazebo>
+    <gazebo>
+    <plugin name="gazebo_ros_diff_drive" filename="libgazebo_ros_diff_drive.so">
+      <!-- Update rate in Hz -->
+      <update_rate>10</update_rate>
+      <!-- wheels -->
+      <left_joint>base_left_wheel_joint</left_joint>
+      <right_joint>base_right_wheel_joint</right_joint>
+      <!-- kinematics -->
+      <wheel_separation>0.45</wheel_separation>
+      <wheel_diameter>0.2</wheel_diameter>
+      <!-- input -->
+      <!-- <command_topic>cmd_vel</command_topic> -->
+      <!-- output -->
+      <publish_odom>true</publish_odom>
+      <publish_odom_tf>true</publish_odom_tf>
+      <publish_wheel_tf>true</publish_wheel_tf>
+      <odometry_topic>odom</odometry_topic>
+      <odometry_frame>odom</odometry_frame>
+      <robot_base_frame>ground</robot_base_frame>
+    </plugin>
+    </gazebo>
 </robot>

Commit message: add lidar and maps

File: src/my_robot_description/urdf/my_robot.urdf.xacro (robot description, xacro)
@@ -4,4 +4,5 @@
     <xacro:include filename="simple_robot_car.urdf.xacro"/>
     <xacro:include filename="simple_robot_car_gazebo.urdf.xacro"/>
-    <xacro:include filename="camera.xacro"/>
+    <!-- <xacro:include filename="camera.xacro"/> -->
+    <xacro:include filename="lidar.xacro"/>
 </robot>

File: src/my_robot_description/urdf/simple_robot_car.urdf (robot description, URDF)
Before this commit: robot my_robot, 5 links, 4 joints
Links:
- removed link ground
- added link base_footprint
Joints:
- removed joint ground_base_joint
- added joint base_footprint_base_joint: type fixed, parent base_footprint, child base_link, origin xyz=0 0 0.05 rpy=0 0 0

File: src/my_robot_description/urdf/simple_robot_car.urdf.xacro (robot description, xacro)
@@ -24,5 +24,5 @@
         </link>
     </xacro:macro>
-    <link name="ground">
+    <link name="base_footprint">
     </link>
     <link name="base_link">
@@ -62,6 +62,6 @@
                                 xyz="0 0 0" rpy="0 0 0" />
     </link>
-    <joint name="ground_base_joint" type="fixed">
-        <parent link="ground" />
+    <joint name="base_footprint_base_joint" type="fixed">
+        <parent link="base_footprint" />
         <child link="base_link" />
         <origin xyz="0 0 ${wheel_radius}" rpy="0 0 0" />

File: src/my_robot_description/urdf/simple_robot_car_gazebo.urdf.xacro (robot description, xacro)
@@ -33,5 +33,5 @@
         <odometry_topic>odom</odometry_topic>
         <odometry_frame>odom</odometry_frame>
-        <robot_base_frame>ground</robot_base_frame>
+        <robot_base_frame>base_footprint</robot_base_frame>
         </plugin>
     </gazebo>
