Commit message: update file

File: src/my_robot_description/urdf/lidar.xacro (robot description, xacro)
@@ -1,7 +1,7 @@
 <?xml version="1.0"?>
 <robot xmlns:xacro="http://www.ros.org/wiki/xacro">
-    <xacro:property name="lidar_length" value="0.1"/>
-    <xacro:property name="lidar_width" value="0.1"/>
-    <xacro:property name="lidar_height" value="0.1"/>
+    <xacro:property name="lidar_length" value="0.01"/>
+    <xacro:property name="lidar_width" value="0.01"/>
+    <xacro:property name="lidar_height" value="0.01"/>
     <link name="lidar_link">
         <visual>
@@ -10,4 +10,5 @@
             </geometry>
             <material name="grey"/>
+            <origin xyz="0 0 ${lidar_height / 2.0}" rpy="0 0 0"></origin>
         </visual>
         <collision>

File: src/my_robot_description/urdf/my_robot.urdf.xacro (robot description, xacro)
@@ -2,5 +2,6 @@
 <robot name="my_robot" xmlns:xacro="http://www.ros.org/wiki/xacro">
     <xacro:include filename="common_properties.xacro" />
-    <xacro:include filename="simple_robot_car.urdf.xacro"/>
+    <!-- <xacro:include filename="simple_robot_car.urdf.xacro"/> -->
+    <xacro:include filename="vacuum_robot_base.xacro"/>
     <xacro:include filename="simple_robot_car_gazebo.urdf.xacro"/>
     <!-- <xacro:include filename="camera.xacro"/> -->

File: src/my_robot_description/urdf/vacuum_robot_base.xacro (robot description, xacro)
@@ -2,5 +2,4 @@
 <robot xmlns:xacro="http://www.ros.org/wiki/xacro">
     <xacro:property name="base_length" value="0.3" />
-    <xacro:property name="base_width" value="0.3" />
     <xacro:property name="base_height" value="0.1" />
     <xacro:property name="wheel_radius" value="0.05" />
@@ -29,5 +28,5 @@
         <visual>
             <geometry>
-                <box size="${base_length} ${base_width} ${base_height}" />
+                <cylinder radius="${base_length / 2.0}" length="${base_height}" />
             </geometry>
             <origin xyz="0 0 ${base_height / 2.0}" rpy="0 0 0"></origin>
@@ -36,10 +35,9 @@
         <collision>
             <geometry>
-                <box size="${base_length} ${base_width} ${base_height}" />
+                <cylinder radius="${base_length}" length="${base_height}" />
             </geometry>
             <origin xyz="0 0 ${base_height / 2.0}" rpy="0 0 0"></origin>
         </collision>
-        <xacro:box_inertia  m="5.0" l="${2*base_length}" w="${2*base_width}"  h="${2*base_height}"
-                            xyz="0 0 ${base_height / 2.0}" rpy="0 0 0" />
+        <xacro:cylinder_inertia m="5.0" r="${2*base_length}" h="${2*base_height}" xyz="0 0 0" rpy="0 0 0" />
     </link>
     <xacro:wheel_link prefix="right" />
@@ -70,5 +68,5 @@
         <parent link="base_link" />
         <child link="right_wheel_link" />
-        <origin xyz="${-base_length*0 / 4.0} ${-base_width / 2.0 - wheel_length / 2.0} 0" rpy="0 0 0" />
+        <origin xyz="0 ${-base_length / 2.0 - wheel_length / 2.0} 0" rpy="0 0 0" />
         <axis xyz="0 1 0" />
     </joint>
@@ -76,5 +74,5 @@
         <parent link="base_link" />
         <child link="left_wheel_link" />
-        <origin xyz="${-base_length*0 / 4.0} ${base_width / 2.0 + wheel_length / 2.0} 0" rpy="0 0 0" />
+        <origin xyz="0 ${base_length / 2.0 + wheel_length / 2.0} 0" rpy="0 0 0" />
         <axis xyz="0 1 0" />
     </joint>
