Commit message: update

File: src/my_robot_description/urdf/vacuum_robot_base.xacro (robot description, xacro)
@@ -68,5 +68,5 @@
         <parent link="base_link" />
         <child link="right_wheel_link" />
-        <origin xyz="0 ${-base_length / 2.0 - wheel_length / 2.0} 0" rpy="0 0 0" />
+        <origin xyz="0 ${-base_length / 2.0 + wheel_length / 2.0} 0" rpy="0 0 0" />
         <axis xyz="0 1 0" />
     </joint>
@@ -74,5 +74,5 @@
         <parent link="base_link" />
         <child link="left_wheel_link" />
-        <origin xyz="0 ${base_length / 2.0 + wheel_length / 2.0} 0" rpy="0 0 0" />
+        <origin xyz="0 ${base_length / 2.0 - wheel_length / 2.0} 0" rpy="0 0 0" />
         <axis xyz="0 1 0" />
     </joint>
